Commit message: Single robot isolated and working

File: src/simulation/urdf/sam_bot.urdf (robot description, URDF)
Before this commit: robot sam_bot, 5 links, 4 joints
Links:
- removed link base_footprint
- removed link base_link
- removed link gnss_link
- removed link imu_link
- removed link lidar_link
- added link pippo/base_footprint
- added link pippo/base_link; collision box size=${base_length} ${base_width} ${base_height}; visual box size=${base_length} ${base_width} ${base_height}
- added link pippo/gnss_link, mass 0.005; collision sphere radius=0.05; visual sphere radius=0.05
- added link pippo/imu_link; collision box size=0.1 0.1 0.1; visual box size=0.1 0.1 0.1
- added link pippo/lidar_link, mass 0.125; collision cylinder length=0.055 radius=0.0508; visual cylinder length=0.055 radius=0.0508
Joints:
- joint base_joint: child base_footprint -> pippo/base_footprint; parent base_link -> pippo/base_link
- joint gnss_joint: child gnss_link -> pippo/gnss_link; parent base_link -> pippo/base_link
- joint imu_joint: child imu_link -> pippo/imu_link; parent base_link -> pippo/base_link
- joint lidar_joint: child lidar_link -> pippo/lidar_link; parent base_link -> pippo/base_link
