Commit message: multi-robot cmd_vel working

File: src/simulation/urdf/pluto.urdf (robot description, URDF)
Before this commit: robot pippo, 5 links, 4 joints
Links:
- removed link pippo/base_footprint
- removed link pippo/base_link
- removed link pippo/gnss_link
- removed link pippo/imu_link
- removed link pippo/lidar_link
- added link pluto/base_footprint
- added link pluto/base_link; collision box size=${base_length} ${base_width} ${base_height}; visual box size=${base_length} ${base_width} ${base_height}
- added link pluto/gnss_link, mass 0.005; collision sphere radius=0.05; visual sphere radius=0.05
- added link pluto/imu_link; collision box size=0.1 0.1 0.1; visual box size=0.1 0.1 0.1
- added link pluto/lidar_link, mass 0.125; collision cylinder length=0.055 radius=0.0508; visual cylinder length=0.055 radius=0.0508
Joints:
- joint base_joint: child pippo/base_footprint -> pluto/base_footprint; parent pippo/base_link -> pluto/base_link
- joint gnss_joint: child pippo/gnss_link -> pluto/gnss_link; parent pippo/base_link -> pluto/base_link
- joint imu_joint: child pippo/imu_link -> pluto/imu_link; parent pippo/base_link -> pluto/base_link
- joint lidar_joint: child pippo/lidar_link -> pluto/lidar_link; parent pippo/base_link -> pluto/base_link
